Commit message: teleop_gen3_mujoco

File: assets/arx/Gen/GEN3-6DOF.urdf (robot description, URDF)
Before this commit: robot GEN3-6DOF_VISION_URDF_ARM_V01, 11 links, 10 joints
Links:
- link base_link: geometry collision mesh filename=D:/xrobotics/XRoboToolkit-Teleop-Sample-Python/assets/arx/G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; visual mesh filename=D:/xrobotics/XRoboToolkit-Teleop-Sample-Python/assets/arx/G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
- link bicep_link: geometry collision mesh filename=D:/xrobotics/XRoboToolkit-Teleop-Sample-Python/assets/arx/G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; visual mesh filename=D:/xrobotics/XRoboToolkit-Teleop-Sample-Python/assets/arx/G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
- link bracelet_link: geometry collision mesh filename=D:/xrobotics/XRoboToolkit-Teleop-Sample-Python/assets/arx/G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; visual mesh filename=D:/xrobotics/XRoboToolkit-Teleop-Sample-Python/assets/arx/G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
- link forearm_link: geometry collision mesh filename=D:/xrobotics/XRoboToolkit-Teleop-Sample-Python/assets/arx/G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; visual mesh filename=D:/xrobotics/XRoboToolkit-Teleop-Sample-Python/assets/arx/G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
- link shoulder_link: geometry collision mesh filename=D:/xrobotics/XRoboToolkit-Teleop-Sample-Python/assets/arx/G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; visual mesh filename=D:/xrobotics/XRoboToolkit-Teleop-Sample-Python/assets/arx/G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
- link spherical_wrist_1_link: geometry collision mesh filename=D:/xrobotics/XRoboToolkit-Teleop-Sample-Python/assets/arx/G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; visual mesh filename=D:/xrobotics/XRoboToolkit-Teleop-Sample-Python/assets/arx/G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
- link spherical_wrist_2_link: geometry collision mesh filename=D:/xrobotics/XRoboToolkit-Teleop-Sample-Python/assets/arx/G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; visual mesh filename=D:/xrobotics/XRoboToolkit-Teleop-Sample-Python/assets/arx/G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

Commit message: gen3 urdf

File: assets/arx/Gen/GEN3-6DOF.urdf (robot description, URDF)
Before this commit: robot GEN3-6DOF, 11 links, 10 joints
Links:
- removed link camera_color_frame
- removed link camera_depth_frame
- removed link camera_link
- removed link end_effector_link
- link base_link: geometry collision mesh filename=meshes/base_link.STL; visual mesh filename=meshes/base_link.STL
- link bicep_link: geometry collision mesh filename=meshes/bicep_link.STL; visual mesh filename=meshes/bicep_link.STL
- link bracelet_link: geometry collision mesh filename=meshes/bracelet_with_vision_link.STL; visual mesh filename=meshes/bracelet_with_vision_link.STL
- link forearm_link: geometry collision mesh filename=meshes/forearm_link.STL; visual mesh filename=meshes/forearm_link.STL
- link shoulder_link: geometry collision mesh filename=meshes/shoulder_link.STL; visual mesh filename=meshes/shoulder_link.STL
- link spherical_wrist_1_link: geometry collision mesh filename=meshes/spherical_wrist_1_link.STL; visual mesh filename=meshes/spherical_wrist_1_link.STL
- link spherical_wrist_2_link: geometry collision mesh filename=meshes/spherical_wrist_2_link.STL; visual mesh filename=meshes/spherical_wrist_2_link.STL
Joints:
- removed joint camera_module
- removed joint color_module
- removed joint depth_module
- removed joint end_effector
- joint joint_1: limit effort=39 velocity=1.3963 -> lower=-3.14 upper=3.14 effort=39 velocity=1.3963; type continuous -> revolute
- joint joint_4: limit effort=9 velocity=1.2218 -> lower=-3.14 upper=3.14 effort=9 velocity=1.2218; type continuous -> revolute
- joint joint_6: limit effort=9 velocity=1.2218 -> lower=-3.14 upper=3.14 effort=9 velocity=1.2218; type continuous -> revolute

Commit message: gen3

File: assets/arx/Gen/GEN3-6DOF.urdf (robot description, URDF)
Before this commit: robot GEN3-6DOF, 7 links, 6 joints
Joints:
- joint joint_1: limit lower=-3.14 upper=3.14 effort=39 velocity=1.3963 -> lower=-3.14 upper=3.14 effort=99 velocity=1.3963
