Commit message: gen3

File: assets/arx/Gen/GEN3-7DOF.urdf (robot description, URDF)
Before this commit: robot GEN3-7DOF_BRAKES_VISION_URDF_ARM_V01, 8 links, 7 joints
Joints:
- joint joint_1: limit lower=-3.14 upper=3.14 effort=39 velocity=1.3963 -> (none); type revolute -> continuous
- joint joint_3: limit lower=-3.14 upper=3.14 effort=39 velocity=1.3963 -> (none); type revolute -> continuous
- joint joint_5: limit lower=-3.14 upper=3.14 effort=9 velocity=1.2218 -> (none); type revolute -> continuous
- joint joint_7: limit lower=-3.14 upper=3.14 effort=9 velocity=1.2218 -> (none); type revolute -> continuous
